File: THERMOMeter/HW/V1_09122022/1- Design Files/_THERMOMeter_/[2] - BLOCK DIAGRAM.kicad_sch (KiCad schematic)
At the start: 0 parts

Commit message: thermometer main schematic has been done
Other:
- note added: "7SEGMENTS 4 DIGITS"
- note removed: "7SEGMENTS 2 X 2DIGITS RED AND GREEN"
Changed lines of the file:
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@@
     (effects (font (size 5 5)) (justify left bottom))
   )
-  (text "7SEGMENTS\n2 X 2DIGITS\nRED AND GREEN" (at 328.93 106.68 0)
+  (text "7SEGMENTS\n4 DIGITS" (at 334.01 106.68 0)
     (effects (font (size 3 3)) (justify left bottom))
   )

Commit message: hardware template has been modified
Other:
- company: (none) -> Siavash Taher Parvar
- title: (none) -> Thermo Meter
Changed lines of the file:
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@@
 (kicad_sch (version 20211123) (generator eeschema)
   (paper "B")
+  (title_block
+    (title "Thermo Meter")
+    (company "Siavash Taher Parvar")
+    (comment 1 "Siavash Taher Parvar")
+    (comment 2 "Siavash Taher Parvar")
+    (comment 3 "Siavash Taher Parvar")
+    (comment 8 "No Variant")
+    (comment 9 "N/A")
+  )
   (polyline (pts (xy 130.81 135.89) (xy 189.23 135.89))
     (stroke (width 0) (type default) (color 0 0 0 0))
