File: THERMOMeter/HW/V1_09122022/1- Design Files/_THERMOMeter_/[3] - MAIN SCHEMATIC.kicad_sch (KiCad schematic)
At the start: 10 parts

Commit message: thermometer main schematic has been done
Parts:
- added C? (x3): 100nF, symbol THERMOMeter_LIB:100nF
- added C? (x2): 1uF, symbol THERMOMeter_LIB:1uF
- added D?: LED_RED, symbol THERMOMeter_LIB:LED_RED
- added DIS?: LDQ-M282RI, symbol THERMOMeter_LIB:LDQ-M282RI
- added J? (x2): XH_CONN_2POS_RA, symbol THERMOMeter_LIB:XH_CONN_2POS_RA
- added J?: USBB_RECEPT_RA, symbol THERMOMeter_LIB:USBB_RECEPT_RA
- added J?: MHDR_6POS_VERT, symbol THERMOMeter_LIB:MHDR_6POS_VERT
- added LS?: CMI-9653S-SMT-TR, symbol THERMOMeter_LIB:CMI-9653S-SMT-TR
- added R? (x9): 470R, symbol THERMOMeter_LIB:470R
- added R?: 2KR, symbol THERMOMeter_LIB:2KR
- added R?: 4K7R, symbol THERMOMeter_LIB:4K7R
- added R? (x2): 10KR, symbol THERMOMeter_LIB:10KR
- added TC? (x2): 4u7F/10V, symbol THERMOMeter_LIB:4u7F/10V
- added U? (x2): SN74HCS595BQBR, symbol THERMOMeter_LIB:SN74HCS595BQBR
- added U? (x2): TC7SZ34FU,LJ(CT, symbol THERMOMeter_LIB:TC7SZ34FU,LJ(CT
- added U?: MCP73832T-2DCI/OT, symbol THERMOMeter_LIB:MCP73832T-2DCI/OT
Connections:
- net GND: now also C?.1, C?.1, C?.1, C?.1, C?.1, J?.2, J?.2, J?.4 (ID), J?.5 (GND), J?.6, LS?.2 (-), R?.1, TC?.1, TC?.1, U?. (VSS), U?.13 (/OE), U?.13 (/OE), U?.3 (GND), U?.3 (GND), U?.8 (GND), U?.8 (GND)
- net MOSI: now reaches U?.6 ((MOSI/AIN0/OC0A/PCINT0)_PB0)
- net MOSI: now also J?.1, U?.2 (INA)
- net MISO: now reaches U?.7 ((MISO/AIN1/OC0B/INT0/PCINT1)_PB1)
- net MISO: now also J?.2, U?.14 (SER)
- net SCK: now reaches U?.9 ((SCK/ADC1/T0/PCINT2)_PB2)
- net SCK: now also J?.2, R?.1, J?.3
- net +3.3V renamed +BATT
- net +BATT: now also C?.2, C?.2, C?.2, C?.2, C?.2, J?.1, R?.2, R?.2, R?.2, TC?.2, U?.16 (VCC), U?.16 (VCC), U?.3 (VBAT), U?.5 (VCC), U?.5 (VCC)
- net RST renamed RESET
- net RESET: now also J?.4
- removed net TEMP_1WIRE: J?.2, R?.1, U?.2 ((PCINT3/CLKI/ADC3)_PB3)
- new net: R?.1, U?.2 (QC)
- new net: DIS?.4 (C), R?.2
- new net: R?.2, U?.5 (PROG)
- new net: LS?.1 (+), U?.4 (OUT_Y)
- new net: R?.1, U?.7 (QH)
- new net: DIS?.3 (DP1), R?.2
- new net: R?.1, U?.6 (QG)
- new net: DIS?.5 (G), R?.2
- new net: DIS?.9 (DIG_2), U?.1 (QB)
- new net: R?.1, U?.10 (/SRCLR) (x2)
- new net: U?.11 (SRCLK), U?.11 (SRCLK), U?.12 (RCLK), U?.12 (RCLK), U?.4 (OUT_Y)
- new net: U?.14 (SER), U?.9 (QH')
- new net: DIS?.12 (DIG_1), U?.15 (QA)
- new net: DIS?.8 (DIG_3), U?.2 (QC)
- new net: DIS?.6 (DIG_4), U?.3 (QD)
- new net: U?.2 (INA), U?.4 (QE)
- new net: R?.1, U?.1 (QB)
- new net: R?.1, U?.15 (QA)
- new net: R?.1, U?.3 (QD)
- new net: R?.1, U?.4 (QE)
- new net: R?.1, U?.5 (QF)
- new net: DIS?.10 (F), R?.2
- new net: DIS?.2 (D), R?.2
- new net: DIS?.7 (B), R?.2
- new net: DIS?.11 (A), R?.2
- new net: D?.2, R?.2
- new net: DIS?.1 (E), R?.2
- new net: R?.1, U?.1 (STAT)
- new net ADC_PTC/NTC: J?.1, R?.1, U?.2 ((PCINT3/CLKI/ADC3)_PB3)
- new net VBUS: D?.1, J?.1 (VCC), TC?.2, U?.4 (VDD)
Other:
- note added: "BATTERY CHARGER"
- note added: "PROGRAMMER CONNECTOR"
- moved on the sheet: C?, J?, R?, U?

Commit message: hardware template has been modified
Other:
- company: (none) -> Siavash Taher Parvar
- title: (none) -> Thermo Meter
Changed lines of the file:
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@@
 (kicad_sch (version 20211123) (generator eeschema)
   (paper "B")
+  (title_block
+    (title "Thermo Meter")
+    (company "Siavash Taher Parvar")
+    (comment 1 "Siavash Taher Parvar")
+    (comment 2 "Siavash Taher Parvar")
+    (comment 3 "Siavash Taher Parvar")
+    (comment 8 "No Variant")
+    (comment 9 "N/A")
+  )
