File: THERMOMeter/HW/V1_09122022/1- Design Files/_THERMOMeter_/[4] - MECHANICAL PARTS.kicad_sch (KiCad schematic)
At the start: 0 parts

Commit message: hardware template has been modified
Other:
- company: (none) -> Siavash Taher Parvar
- title: (none) -> Thermo Meter
Changed lines of the file:
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@@
 (kicad_sch (version 20211123) (generator eeschema)
-  (paper "A4")
+  (paper "B")
+  (title_block
+    (title "Thermo Meter")
+    (company "Siavash Taher Parvar")
+    (comment 1 "Siavash Taher Parvar")
+    (comment 2 "Siavash Taher Parvar")
+    (comment 3 "Siavash Taher Parvar")
+    (comment 8 "No Variant")
+    (comment 9 "N/A")
+  )
 )
