File: FREQMeter/HW/V1_21092022/1- Design Files/_HW_FREQMeter/[03] - MCU_PB.kicad_sch (KiCad schematic)
At the start: 0 parts

Commit message: progress on Frequency meter hardware
Parts:
- added C? (x4): 100nF, symbol FREQMeter:100nF
- added J?: MHDR_6POS_VERT, symbol FREQMeter:MHDR_6POS_VERT
- added R? (x5): 100R, symbol FREQMeter:100R
- added R? (x2): 10KR, symbol FREQMeter:10KR
- added SW?: SPST_NO, symbol FREQMeter:SPST_NO
- added U?: ATTINY13A-MMU, symbol FREQMeter:ATTINY13A-MMU
- added U?: 74LVC3G34GS,115, symbol FREQMeter:74LVC3G34GS,115
Connections:
- new net: C?.2, R?.2, SW?.1, U?.6 (3A)
- new net: R?.1, U?.4 ((PCINT4/ADC2)_PB4)
- new net: R?.1, U?.2 ((PCINT3/CLKI/ADC3)_PB3)
- new net GND: C?.1, C?.1, C?.1, C?.1, J?.1, R?.1, U?.4 (GND), U?.5 (GND)
- new net INPUT_SIG: R?.2
- new net MCU_RESET: C?.2, J?.3, R?.1, U?.1 (RESET)
- new net MISO: J?.5, R?.1, U?.7 ((MISO/AIN1/OC0B/INT0/PCINT1)_PB1)
- new net MOSI: J?.6, R?.1, U?.6 ((MOSI/AIN0/OC0A/PCINT0)_PB0)
- new net PUSH_BUTTON: R?.2, U?.2 (3Y)
- new net SCK: J?.4, R?.1, U?.9 ((SCK/ADC1/T0/PCINT2)_PB2)
- new net SR_7SEG_DATA: R?.2
- new net SR_CLK: R?.2, U?.1 (1A), U?.3 (2A)
- new net SR_CNTR_DATA: R?.2
- new net SR_SCHP_CLK: U?.7 (1Y)
- new net SR_STCP_CLK: U?.5 (2Y)
- new net VCC: C?.2, C?.2, R?.2, SW?.2, U?.10 (VCC), U?.8 (VCC)
Other:
- note added: "INFO:"
- note added: "PROGRAMMER CONN"

Commit message: frequency meter input schematic in progress
Changed lines of the file:
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@@
     (stroke (width 0) (type default) (color 0 0 0 0))
   )
-  (wire (pts (xy 194.31 128.27) (xy 201.93 128.27))
+  (wire (pts (xy 194.31 128.27) (xy 219.71 128.27))
     (stroke (width 0) (type default) (color 0 0 0 0))
   )
@@
     (effects (font (size 1.27 1.27)) (justify left bottom))
   )
-  (label "INPUT_SIG" (at 201.93 128.27 0)
-    (effects (font (size 1.27 1.27)) (justify left bottom))
-  )
   (label "MOSI" (at 121.92 181.61 0)
     (effects (font (size 1.27 1.27)) (justify left bottom))
@@
     (effects (font (size 1.27 1.27)) (justify left))
   )
+  (hierarchical_label "INPUT_SIG" (shape input) (at 219.71 128.27 0)
+    (effects (font (size 1.27 1.27)) (justify left))
+  )
