File: FREQMeter/HW/V1_21092022/1- Design Files/_HW_FREQMeter/[04] - SIG INPUT.kicad_sch (KiCad schematic)
At the start: 0 parts

Commit message: frequency meter input schematic in progress
Parts:
- added C? (x2): 10pF, symbol FREQMeter:10pF
- added C? (x3): 1uF, symbol FREQMeter:1uF
- added C? (x3): 100nF, symbol FREQMeter:100nF
- added J?: BNC_CONN_RA, symbol FREQMeter:BNC_CONN_RA
- added R? (x2): 15K8R, symbol FREQMeter:15K8R
- added R?: 22R, symbol FREQMeter:22R
- added R?: 47KR, symbol FREQMeter:47KR
- added R? (x2): 100R, symbol FREQMeter:100R
- added R? (x2): 120R, symbol FREQMeter:120R
- added R?: 10KR, symbol FREQMeter:10KR
- added R?: 50R, symbol FREQMeter:50R
- added U? (x4): TLV3541IDBVR, symbol FREQMeter:TLV3541IDBVR
- added U? (x2): SN74HCS125BQAR, symbol FREQMeter:SN74HCS125BQAR
Connections:
- new net: C?.1, R?.1, R?.2
- new net: C?.2, R?.1, U?.1, U?.4 (-IN)
- new net: R?.1, R?.2 (x2)
- new net: C?.2, R?.2, U?.3 (+IN)
- new net: R?.2, U?.3 (1Y)
- new net: R?.2, U?.2 (1A)
- new net: R?.1, R?.2, U?.4 (-IN)
- new net: R?.1, R?.2, U?.1
- new net: R?.2, U?.3 (+IN)
- new net: J?.1, R?.1, R?.2
- new net GND: C?.1, C?.1, C?.1, C?.1, C?.1, C?.1, C?.1, J?.2, R?.1, R?.1, U?.2 (V-), U?.2 (V-), U?.7-UD (GND)
- new net INPUT_SIG: R?.1
- new net VCC: C?.2, C?.2, C?.2, C?.2, C?.2, C?.2, U?.12 (1A), U?.13 (1~{OE}), U?.14-UD (VCC), U?.5 (V+), U?.5 (V+)
- new net X1000_PWR: U?.1 (1~{OE})
Other:
- note added: "74HCS125"
- note added: "BUFFER"
- note added: "DESIGN & LAYOUT NOTE:"
- note added: "DNF"
- note added: "INFO:"
- note added: "INPUT AND MATCHING CIRCUIT"
- note added: "LAYOUT NOTE:"
- note added: "LPF Sallen-Key Filter"
- note added: "OPEN-LOOP Filter"
- note added: "f0 = 1.000 MHz Q = 0.5 G = 1"
- note added: "• Noise propagates into analog circuitry through the power pins of the circuit as a whole and the operational amplifier. Use bypass capacitors to reduce the coupled noise by providing low-impedance power sources local to the analog circuitry. - Connect low-ESR, 0.1-μF ceramic bypass capacitors between each supply pin and ground, placed as close to the device as possible. A single bypass capacitor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"

Commit message: Input signal schematic has been modified
Parts:
- removed R?: 47KR, symbol FREQMeter:47KR
- removed R?: 100R, symbol FREQMeter:100R
- removed R?: 10KR, symbol FREQMeter:10KR
- added C?: 10pF, symbol FREQMeter:10pF
- added R?: 470KR, symbol FREQMeter:470KR
- added R?: 120R, symbol FREQMeter:120R
- added R?: 100KR, symbol FREQMeter:100KR
- added R?: 15K8R, symbol FREQMeter:15K8R
- added R?: 1MR, symbol FREQMeter:1MR
Connections:
- net GND: now also C?.1, R?.1
- net INPUT_SIG: now also J?.1, R?.2, R?.1
- net at C?.2, U?.1, U?.4 (-IN): now also R?.1
- net at U?.4 (-IN): now also R?.1, R?.2
- net at R?.1: now also C?.2, R?.2; no longer U?.1
- net at U?.3 (+IN): now also R?.2
- new net: R?.1, R?.2, U?.1
- new net: R?.1, R?.2
Other:
- note removed: "DNF"
- note removed: "OPEN-LOOP Filter"
- moved on the sheet: C?, J?, R?, U?A, U?B, U?D
